File: platform/kicad/peripheral_hat/peripheral_hat.kicad_pcb (KiCad board)
At the start: 2 copper layers, 30 x 65 mm, 32 parts, among them J1 CRJ032-1-TH, J2 Pi Header, T1 PT61018PEL, U2 ENC28J60x-SS, U3 AP63205WU-7, Y1 ABLS-25.000MHZ-20-A4-F-T

Commit message: Peripheral PCB: Finalise for production
Parts:
- removed Y1: ABLS-25.000MHZ-20-A4-F-T, AusOcean:XTAL_ABLS-25.000MHZ-20-A4-F-T
- added G***: LOGO, LOGO, F.Cu at (199.9, 96.3)
- added X1: ~, AusOcean:X322525MOB4SI, F.Cu at (208.4, 106.2)
- moved C15 2.78 mm to (206.2, 110.1), turned to -90 degrees
- moved C16 2.05 mm to (206.2, 105.0), turned to -90 degrees
- moved L1 1.36 mm to (194.2, 87.8)
Routing:
- net Net-(U2-OSC1): track 14.4 -> 3.00 mm
- net Net-(U2-OSC2): track 14.1 -> 3.01 mm
- net GND: track 3.10 -> 0.00 mm
- net +5V: track 28.4 -> 29.3 mm
- added copper zone on F.Cu, net Net-(U2-OSC1)
- added copper zone on F.Cu, net Net-(U2-OSC2)
Other:
- board text added: "PoE Hat"
- board text added: "PoE IN"
- board text added: "david@ausocean.org"
- board text added: "v1 revA"

Commit message: WIP
Parts:
- removed U3: AP63205WU-7, AusOcean:SOIC_05WU-7_DIO
- removed X1: ~, AusOcean:X322525MOB4SI
- added C17: 4.7nF, Capacitor_SMD:C_0402_1005Metric, F.Cu at (202.5, 104.1)
- added C18: 1.5nF, Capacitor_SMD:C_0402_1005Metric, F.Cu at (203.5, 104.1)
- added C19: 4.7nF, Capacitor_SMD:C_0402_1005Metric, F.Cu at (209.6, 117.0)
- added C20: 100nF, Capacitor_SMD:C_0402_1005Metric, F.Cu at (194.9, 94.0)
- added C21: 10uF, Capacitor_SMD:C_1206_3216Metric, F.Cu at (207.8, 89.2)
- added C22: 100nF, Capacitor_SMD:C_0603_1608Metric, F.Cu at (210.4, 89.7)
- added C23: 22uF, Capacitor_SMD:C_1206_3216Metric, F.Cu at (201.0, 86.4)
- added C24: 22uF, Capacitor_SMD:C_1206_3216Metric, F.Cu at (201.0, 83.9)
- added D1: APT1608LZGCK, Capacitor_SMD:C_0805_2012Metric, F.Cu at (210.0, 97.8)
- added FB2: MMZ1608B121CTAH0, Capacitor_SMD:C_0603_1608Metric, F.Cu at (207.4, 115.5)
- added FB3: MMZ1608B121CTAH0, Capacitor_SMD:C_0603_1608Metric, F.Cu at (207.4, 117.2)
- added J3: Pogo Pin, AusOcean:YZ70115093P-02, B.Cu at (210.8, 120.4)
- added J4: Pogo Pin, AusOcean:YZ70115093P-02, B.Cu at (210.8, 122.5)
- added R1: 49.9, Resistor_SMD:R_0402_1005Metric, F.Cu at (190.6, 123.4)
- added R2: 49.9, Resistor_SMD:R_0402_1005Metric, F.Cu at (190.6, 121.3)
- added R3: 49.9, Resistor_SMD:R_0402_1005Metric, F.Cu at (206.6, 121.3)
- added U1: LAN9500A-ABZJ, AusOcean:QFN56_8X8MC_MCH, F.Cu at (199.0, 109.9)
- added XTAL1: SIT1602AI-32-33E-25.000000Y, AusOcean:SON4_SIT1602-3_SIT, F.Cu at (208.0, 110.1)
- C1: value 10u -> 1nF 2KV; footprint Capacitor_SMD:C_1206_3216Metric -> Capacitor_SMD:C_0402_1005Metric
- C10, C7, C8: value 0.1uF -> 100nF; footprint Capacitor_SMD:C_0201_0603Metric -> Capacitor_SMD:C_0402_1005Metric
- C11, C12: value 0.1uF -> 4.7nF; footprint Capacitor_SMD:C_0201_0603Metric -> Capacitor_SMD:C_0402_1005Metric; moved to B.Cu
- C13: value 0.1uF -> 1.5nF; footprint Capacitor_SMD:C_0201_0603Metric -> Capacitor_SMD:C_0402_1005Metric; moved to B.Cu
- C14: value 0.1uF -> 4.7nF; footprint Capacitor_SMD:C_0201_0603Metric -> Capacitor_SMD:C_0402_1005Metric
- C15: value 20pF -> 1uF; footprint Capacitor_SMD:C_0201_0603Metric -> Capacitor_SMD:C_0402_1005Metric; moved to B.Cu
- C16: value 20pF -> 100nF; footprint Capacitor_SMD:C_0201_0603Metric -> Capacitor_SMD:C_0402_1005Metric; moved to B.Cu
- C2: value 0.1u -> 22nF; footprint Capacitor_SMD:C_0603_1608Metric -> Capacitor_SMD:C_0402_1005Metric
- C3: value 0.1u -> 100nF; footprint Capacitor_SMD:C_0603_1608Metric -> Capacitor_SMD:C_0402_1005Metric
- C4: value 22u -> 100nF; footprint Capacitor_SMD:C_1206_3216Metric -> Capacitor_SMD:C_0402_1005Metric; moved to B.Cu
- C5: value 22u -> 4.7nF; footprint Capacitor_SMD:C_1206_3216Metric -> Capacitor_SMD:C_0402_1005Metric; moved to B.Cu
- C6: value 0.1uF -> 1.5nF; footprint Capacitor_SMD:C_0201_0603Metric -> Capacitor_SMD:C_0402_1005Metric
- C9: value 0.1uF -> 100nF; footprint Capacitor_SMD:C_0201_0603Metric -> Capacitor_SMD:C_0402_1005Metric; moved to B.Cu
- FB1: value FerriteBead_Small -> MMZ1608B121CTAH0; footprint Resistor_SMD:R_0603_1608Metric -> Capacitor_SMD:C_0603_1608Metric
- L1: value 4.7u -> 4.7uF; footprint AusOcean:WE-XHMI_6060 -> Inductor_SMD:L_Changjiang_FXL0630
- R10: value 2.32k 1% -> 4k7; footprint Resistor_SMD:R_0201_0603Metric -> Resistor_SMD:R_0402_1005Metric
- R11: value 10M -> 33; footprint Resistor_SMD:R_0201_0603Metric -> Resistor_SMD:R_0402_1005Metric
- R4: footprint Resistor_SMD:R_0201_0603Metric -> Resistor_SMD:R_0402_1005Metric
- R5: value 49.9 -> 330; footprint Resistor_SMD:R_0201_0603Metric -> Resistor_SMD:R_0402_1005Metric
- R6, R7: value 49.9 -> 75; footprint Resistor_SMD:R_0201_0603Metric -> Resistor_SMD:R_0402_1005Metric
- R8: value 75 -> 12K 1%; footprint Resistor_SMD:R_0201_0603Metric -> Resistor_SMD:R_0402_1005Metric
- R9: value 75 -> 12K 1%; footprint Resistor_SMD:R_0201_0603Metric -> Resistor_SMD:R_0402_1005Metric; moved to B.Cu
- U2: value ENC28J60x-SS -> AP63205WU-7; footprint Package_SO:SSOP-28_5.3x10.2mm_P0.65mm -> AusOcean:SOIC_05WU-7_DIO
- moved G*** 66.5 mm to (266.4, 98.2)
- moved C1 38.7 mm to (206.6, 127.7), turned to 180 degrees
- moved C2 33.7 mm to (208.7, 123.3), turned to 0 degrees
- moved C5 25.9 mm to (201.1, 109.7), turned to 180 degrees
- moved C4 25.3 mm to (200.3, 112.2), turned to 90 degrees
- moved R5 24.2 mm to (210.0, 95.0)
- moved C3 23.0 mm to (200.1, 116.0), turned to 0 degrees
- moved R10 18.8 mm to (211.4, 110.1), turned to -90 degrees
- moved U2 18.5 mm to (203.8, 91.1), turned to 180 degrees
- moved C13 17.9 mm to (196.7, 112.2), turned to 0 degrees
- moved FB1 16.1 mm to (204.9, 104.7), turned to -90 degrees
- moved R9 15.8 mm to (199.2, 112.2), turned to -90 degrees
- moved C14 14.8 mm to (204.4, 114.3), turned to 90 degrees
- moved R6 14.2 mm to (206.6, 125.1), turned to 0 degrees
- moved R7 12.9 mm to (206.6, 126.4), turned to 0 degrees
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Connections:
- C1 pad 1: 24V -> Net-(C1-Pad1)
- C11 pad 1: Net-(T1-CT1) -> +3V3
- C12 pad 1: Net-(C12-Pad1) -> +3V3
- C13 pad 1: Net-(C13-Pad1) -> +3V3
- C14 pad 1: Net-(U2-VCAP) -> VDDUSBPLL
- C15 pad 1: Net-(U2-OSC1) -> VDDCORE
- C16 pad 1: GND -> VDDCORE
- C16 pad 2: Net-(U2-OSC2) -> GND
- C2 pad 1: 24V -> +3.3VA
- C3 pad 1: Net-(U3-BST) -> +3.3VA
- C3 pad 2: Net-(U3-SW) -> GND
- C4 pad 1: +5V -> +3.3VA
- C5 pad 1: +5V -> +3.3VA
- C6 pad 1: +3V3 -> +3.3VA
- FB1 pad 1: Net-(T1-CT1) -> +3V3
- FB1 pad 2: +3V3 -> +3.3VA
- J2 pad 19: MOSI -> unconnected-(J2-Pin_19-Pad19)
- J2 pad 21: MISO -> unconnected-(J2-Pin_21-Pad21)
- J2 pad 22: INT -> unconnected-(J2-Pin_22-Pad22)
- J2 pad 23: SCK -> unconnected-(J2-Pin_23-Pad23)
- J2 pad 24: CS -> unconnected-(J2-Pin_24-Pad24)
- L1 pad 1: Net-(U3-SW) -> Net-(U2-SW)
- R10 pad 1: GND -> Net-(XTAL1-OE/ST)
- R10 pad 2: Net-(U2-RBIAS) -> +3V3
- R11 pad 1: Net-(U2-OSC2) -> Net-(XTAL1-OUT)
- R11 pad 2: Net-(U2-OSC1) -> XI
- R4 pad 1: Net-(T1-CT1) -> TD-
- R4 pad 2: TPOUT- -> +3.3VA
- R5 pad 1: TPOUT+ -> Net-(D1-A)
- R5 pad 2: Net-(T1-CT1) -> +3V3
- R6 pad 1: TPIN- -> Net-(T1-CT3)
- R6 pad 2: Net-(C12-Pad1) -> Net-(C1-Pad1)
- R7 pad 1: Net-(C12-Pad1) -> Net-(T1-CT4)
- R7 pad 2: TPIN+ -> Net-(C1-Pad1)
- R8 pad 1: Net-(T1-CT3) -> GND
- R8 pad 2: Net-(C13-Pad1) -> USBRBIAS
- R9 pad 1: Net-(T1-CT4) -> GND
- R9 pad 2: Net-(C13-Pad1) -> EXRES
- T1 pad 1: TPOUT+ -> TD+
- T1 pad 2: Net-(T1-CT1) -> +3.3VA
- T1 pad 3: TPOUT- -> TD-
- T1 pad 6: TPIN+ -> RD+
- T1 pad 7: unconnected-(T1-CT2-Pad7) -> +3.3VA
- T1 pad 8: TPIN- -> RD-
- U2 pad 1: Net-(U2-VCAP) -> +5V
- U2 pad 2: GND -> 24V
- U2 pad 3: unconnected-(U2-CLKOUT-Pad3) -> 24V
- U2 pad 4: INT -> GND
- U2 pad 5: unconnected-(U2-~{WOL}-Pad5) -> Net-(U2-SW)
- U2 pad 6: MISO -> Net-(U2-BST)
Routing:
- net 24V: track 0.00 -> 65.5 mm, vias 2 -> 1
- net +3.3VA: track 0.00 -> 58.3 mm, vias 0 -> 8
- net VDDCORE: track 0.00 -> 52.2 mm, vias 0 -> 6
- net GND: track 0.00 -> 19.4 mm, vias 0 -> 18
- net TD-: track 0.00 -> 16.4 mm
- net INT: track 15.6 -> 0.00 mm
- net USBD-: track 0.00 -> 15.2 mm
- net RD+: track 0.00 -> 15.1 mm, vias 0 -> 2
- net TD+: track 0.00 -> 14.9 mm
- net CS: track 14.7 -> 0.00 mm
- net USBD+: track 0.00 -> 13.7 mm, vias 0 -> 1
- net TPIN-: track 13.2 -> 0.00 mm, vias 2 -> 0
- net TPOUT+: track 12.9 -> 0.00 mm, vias 2 -> 0
- net VDDPLL: track 0.00 -> 11.8 mm, vias 0 -> 2
- net RD-: track 0.00 -> 11.8 mm, vias 0 -> 2
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- added copper zone on F.Cu, net +3V3
- added copper zone on B.Cu, net GND
- added copper zone on F.Cu, net Net-(U2-SW)
- removed copper zone on B.Cu, net 24V
- removed copper zone on F.Cu, net Net-(U2-OSC1)
- removed copper zone on F.Cu, net Net-(U2-OSC2)
- removed copper zone on F.Cu, net Net-(U3-SW)
Other:
- outline, holes or cut-outs redrawn
- board text added: "v2 revA"
- board text removed: "v1 revA"
