File: platform/kicad/peripheral_hat/peripheral_hat.kicad_pcb (KiCad board)
At the start: 4 copper layers, 35.5 x 65 mm, 56 parts, among them J1 Pi Header, J4 CRJ032-1-TH, J5 JST EH, J6 JST EH, J7 JST EH, J8 USB_B, T1 PT61018PEL, U1 LAN9500A-ABZJ, U2 AP63205WU-7

Commit message: Peripheral Hat: V2 Rev C
Updates to using a micro-B interface between the pi and the hat.
Parts:
- moved G*** 19.7 mm to (184.7, 88.7)
- moved C17 19.6 mm to (186.0, 109.0)
- moved C1 18.5 mm to (187.6, 108.8), turned to -90 degrees
- moved C19 17.9 mm to (189.0, 110.3)
- moved R9 17.6 mm to (191.5, 110.4), turned to 180 degrees
- moved FB3 17.1 mm to (186.0, 106.5), turned to -90 degrees
- moved FB1 15.7 mm to (187.6, 106.5), turned to 90 degrees
- moved D1 15.4 mm to (197.1, 106.3)
- moved R11 15.4 mm to (197.1, 109.2)
- moved FB2 14.4 mm to (197.3, 91.9), turned to 45 degrees
- moved XTAL1 12.8 mm to (191.5, 107.0), turned to 90 degrees
- moved R2 8.01 mm to (189.6, 93.6), turned to -45 degrees
- moved R1 7.77 mm to (187.6, 100.3), turned to -45 degrees
- moved C12 6.86 mm to (187.9, 99.1), turned to 135 degrees
- moved C7 6.75 mm to (199.2, 103.5), turned to -135 degrees
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Routing:
- net +3V3: track 129.5 -> 114.0 mm, vias 4 -> 1
- net USBD-: track 0.00 -> 11.9 mm
- net USBD+: track 0.00 -> 11.6 mm
- net GND: track 7.42 -> 15.2 mm, vias 82 -> 87
- net NLINK_LED: track 11.6 -> 4.95 mm, vias 2 -> 0
- net VDDPLL: track 12.4 -> 18.3 mm
- net TD-: track 10.8 -> 16.2 mm
- net VDDCORE: track 33.9 -> 29.7 mm, vias 5 -> 3
- net +24V: track 77.2 -> 80.9 mm
- net unconnected-(J1-Pin_19-Pad19): track 3.11 -> 0.00 mm
- net VDDUSBPLL: track 7.09 -> 10.1 mm, vias 2 -> 0
- net +3.3VA: track 55.8 -> 58.6 mm, vias 5 -> 3
- net EXRES: track 5.02 -> 2.68 mm, vias 2 -> 0
- net TD+: track 14.3 -> 16.2 mm
- net Net-(XTAL1-OUT): track 2.05 -> 3.89 mm
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Other:
- board text added: "USB"

Commit message: Try panel
Parts:
- added G***: LOGO, LOGO, B.Cu at (140.4, 78.2)
- added USB1: ZX80-B-5SA(30), lcsc_footprints:C598212_MICRO-USB_SMD_ZX80-B-5SA-30, F.Cu at (139.4, 72.8)
- added USB2: ZX80-B-5SA(30), lcsc_footprints:C598212_MICRO-USB_SMD_ZX80-B-5SA-30, F.Cu at (139.4, 85.4)
Routing:
- net /USB Bridge/D-: track 0.00 -> 12.7 mm
- net /USB Bridge/D+: track 0.00 -> 12.7 mm
- net Net-(USB1-VBUS): track 0.00 -> 12.6 mm
- net Net-(USB1-ID): track 0.00 -> 12.6 mm
- net Net-(USB1-GND-Pad5): track 0.00 -> 12.6 mm
- added copper zone on B.Cu, net Net-(USB1-GND-Pad5)
- added copper zone on F.Cu, net Net-(USB1-GND-Pad5)
- added copper zone on In1.Cu, net Net-(USB1-GND-Pad5)
- added copper zone on In2.Cu, net Net-(USB1-GND-Pad5)
Other:
- board size 35.5 x 65 mm -> 86 x 65 mm
- board text added: "USB Bridge"
- board text added: "v1 revA"
