File: platform/kicad/peripheral_hat/peripheral_hat.kicad_sch (KiCad schematic)
At the start: 43 parts, among them J1 Pi Header, J4 CRJ032-1-TH, T1 PT61018PEL, U1 LAN9500A-ABZJ

Commit message: Try panel
Other:
- added sheet USB Bridge (usb_bridge.kicad_sch)
Changed lines of the file:
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@@
+	)
+	(sheet
+		(at 133.35 173.99)
+		(size 27.94 13.97)
+		(exclude_from_sim no)
+		(in_bom yes)
+		(on_board yes)
+		(dnp no)
+		(fields_autoplaced yes)
+		(stroke
+			(width 0.1524)
+			(type solid)
+		)
+		(fill
+			(color 0 0 0 0)
+		)
+		(property "Sheetname" "USB Bridge"
+			(at 133.35 173.2784 0)
+			(show_name no)
+			(do_not_autoplace no)
+			(effects
+				(font
+					(size 1.27 1.27)
+				)
+				(justify left bottom)
+			)
+		)
+		(property "Sheetfile" "usb_bridge.kicad_sch"
+			(at 133.35 188.5446 0)
+			(hide yes)
+			(show_name no)
+			(do_not_autoplace no)
+			(effects
+				(font
+					(size 1.27 1.27)
+				)
+				(justify left top)
+			)
+		)
+		(instances
+			(project "peripheral_hat"
+				(path "/8dfa5814-59de-42fa-a019-7b76c06633d1"
+					(page "4")
+				)
+			)
+		)
 	)
 	(sheet
