File: platform/kicad/navlight/navlight.kicad_sch (KiCad schematic)
At the start: 8 parts, among them J1 TSL2951, J2 Conn_01x05_Pin

Commit message: Navlight: Update port position
This change reverts the position of the JST to the same side of the
PCB as the lightsensor.

This change also adds the production files to the repo.
Changed lines of the file:
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@@
 (kicad_sch
-	(version 20231120)
+	(version 20250114)
 	(generator "eeschema")
-	(generator_version "8.0")
+	(generator_version "9.0")
 	(paper "A4")
+	(rectangle
+		(start 38.1 38.1)
+		(end 76.2 63.5)
+		(stroke
+			(width 0)
+			(type default)
+		)
+		(fill
+			(type none)
+		)
+	)
+	(rectangle
+		(start 144.78 38.1)
+		(end 182.88 63.5)
+		(stroke
+			(width 0)
+			(type default)
+		)
+		(fill
+			(type none)
+		)
+	)
+	(rectangle
+		(start 104.14 38.1)
+		(end 142.24 63.5)
+		(stroke
+			(width 0)
+			(type default)
+		)
+		(fill
+			(type none)
+		)
+	)
+	(rectangle
+		(start 78.74 38.1)
+		(end 101.6 96.52)
+		(stroke
+			(width 0)
+			(type default)
+		)
+		(fill
+			(type none)
+		)
+	)
+	(text "Mounting"
+		(exclude_from_sim no)
+		(at 56.896 35.814 0)
+		(effects
+			(font
+				(size 2.54 2.54)
+			)
+		)
+	)
+	(text "Photometer"
+		(exclude_from_sim no)
+		(at 124.206 35.56 0)
+		(effects
+			(font
+				(size 2.54 2.54)
+			)
+		)
+	)
+	(text "IO"
+		(exclude_from_sim no)
+		(at 163.322 35.052 0)
+		(effects
+			(font
+				(size 2.54 2.54)
+			)
+		)
+	)
+	(text "Nav Lights"
+		(exclude_from_sim no)
+		(at 89.408 35.306 0)
+		(effects
+			(font
+				(size 2.54 2.54)
+			)
+		)
+	)
 	(junction
 		(at 96.52 76.2)
@@
 			(width 0)
 			(type default)
-		)
-	)
-	(rectangle
-		(start 38.1 38.1)
-		(end 76.2 63.5)
-		(stroke
-			(width 0)
-			(type default)
-		)
-		(fill
-			(type none)
-		)
-	)
-	(rectangle
-		(start 144.78 38.1)
-		(end 182.88 63.5)
-		(stroke
-			(width 0)
-			(type default)
-		)
-		(fill
-			(type none)
-		)
-	)
-	(rectangle
-		(start 104.14 38.1)
-		(end 142.24 63.5)
-		(stroke
-			(width 0)
-			(type default)
-		)
-		(fill
-			(type none)
-		)
-	)
-	(rectangle
-		(start 78.74 38.1)
-		(end 101.6 96.52)
-		(stroke
-			(width 0)
-			(type default)
-		)
-		(fill
-			(type none)
-		)
-	)
-	(text "Mounting"
-		(exclude_from_sim no)
-		(at 56.896 35.814 0)
-		(effects
-			(font
-				(size 2.54 2.54)
-			)
-		)
-	)
-	(text "Photometer"
-		(exclude_from_sim no)
-		(at 124.206 35.56 0)
-		(effects
-			(font
-				(size 2.54 2.54)
-			)
-		)
-	)
-	(text "IO"
-		(exclude_from_sim no)
-		(at 163.322 35.052 0)
-		(effects
-			(font
-				(size 2.54 2.54)
-			)
-		)
-	)
-	(text "Nav Lights"
-		(exclude_from_sim no)
-		(at 89.408 35.306 0)
-		(effects
-			(font
-				(size 2.54 2.54)
-			)
 		)
 	)
@@
 		)
 	)
+	(embedded_fonts no)
 )
